File: hw/pcb/eyevolt.kicad_pcb (KiCad board)
At the start: 4 copper layers, 79 x 45 mm, 21 parts, among them J1 Conn_02x10_Odd_Even, U1 Pico, U2 MCP6L04x-xSL, U3 MCP6L04x-xSL, U4 74HCT4051, U5 MCP6L04x-xSL, U6 MCP6L04x-xSL, U7 74HCT4051

Commit message: First version of PCB completed
Parts:
- removed BT101: 1078, onio_Connector:BAT_1078
- removed H101, H102, H103, H104: Mount-Hole-3.3mm, onio_Mouting-Hole:Mouting-Hole-3.3mm
- added C1: C, Capacitor_SMD:C_0805_2012Metric_Pad1.18x1.45mm_HandSolder, F.Cu at (97.0, 72.0)
- added C2: C, Capacitor_SMD:C_0805_2012Metric_Pad1.18x1.45mm_HandSolder, F.Cu at (98.0, 51.0)
- added C3: C, Capacitor_SMD:C_0805_2012Metric_Pad1.18x1.45mm_HandSolder, F.Cu at (132.1, 61.0)
- added C4: C, Capacitor_SMD:C_0805_2012Metric_Pad1.18x1.45mm_HandSolder, F.Cu at (131.1, 73.5)
- added C5: C, Capacitor_SMD:C_0805_2012Metric_Pad1.18x1.45mm_HandSolder, F.Cu at (132.1, 48.0)
- added C6: C, Capacitor_SMD:C_0805_2012Metric_Pad1.18x1.45mm_HandSolder, F.Cu at (109.0, 51.0)
- added H1: MountingHole_Pad, MountingHole:MountingHole_3.2mm_M3, F.Cu at (151.5, 50.0)
- added H2: MountingHole_Pad, MountingHole:MountingHole_3.2mm_M3, F.Cu at (151.5, 91.0)
- added H3: MountingHole_Pad, MountingHole:MountingHole_3.2mm_M3, F.Cu at (38.5, 91.0)
- added H4: MountingHole_Pad, MountingHole:MountingHole_3.2mm_M3, F.Cu at (38.0, 50.0)
- added J2: Conn_01x15, Connector_PinHeader_2.54mm:PinHeader_1x15_P2.54mm_Vertical, F.Cu at (49.8, 92.0)
- added J3: Conn_01x15, Connector_PinHeader_2.54mm:PinHeader_1x15_P2.54mm_Vertical, F.Cu at (49.8, 87.0)
- U4, U7: footprint Package_SO:SOIC-14_3.9x8.7mm_P1.27mm -> Package_SO:SOIC-16_3.9x9.9mm_P1.27mm
- moved U1 129.6 mm to (61.0, 70.0), turned to 90 degrees
- moved U7 126.6 mm to (97.6, 59.4)
- moved U4 104.4 mm to (97.5, 79.9)
- moved R5 101.4 mm to (120.0, 55.0)
- moved R6 100.8 mm to (120.0, 62.0)
- moved R7 100.6 mm to (120.0, 67.0)
- moved R1 100.2 mm to (120.0, 53.0)
- moved R8 100.2 mm to (120.0, 74.0)
- moved R2 100.0 mm to (120.0, 60.0), turned to 180 degrees
- moved R4 100.0 mm to (120.0, 72.0), turned to 180 degrees
- moved R3 99.9 mm to (120.0, 65.0)
- moved U6 84.1 mm to (131.5, 53.8)
- moved U5 76.7 mm to (131.5, 66.8)
- moved U2 73.4 mm to (108.5, 58.8)
- moved U3 64.0 mm to (131.5, 79.5)
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Connections:
- U1 pad 10: unconnected-(U1-GPIO7-Pad10) -> /WAIT
- U1 pad 11: unconnected-(U1-GPIO8-Pad11) -> /INT
- U1 pad 13: unconnected-(U1-GND-Pad13) -> GND
- U1 pad 14: unconnected-(U1-GPIO10-Pad14) -> /MUX0_S0
- U1 pad 15: unconnected-(U1-GPIO11-Pad15) -> /MUX0_S1
- U1 pad 16: unconnected-(U1-GPIO12-Pad16) -> /MUX0_S2
- U1 pad 17: unconnected-(U1-GPIO13-Pad17) -> /MUX0_EB
- U1 pad 18: unconnected-(U1-GND-Pad18) -> GND
- U1 pad 23: unconnected-(U1-GND-Pad23) -> GND
- U1 pad 24: unconnected-(U1-GPIO18-Pad24) -> /MUX1_EB
- U1 pad 25: unconnected-(U1-GPIO19-Pad25) -> /MUX1_S2
- U1 pad 26: unconnected-(U1-GPIO20-Pad26) -> /MUX1_S1
- U1 pad 27: unconnected-(U1-GPIO21-Pad27) -> /MUX1_S0
- U1 pad 28: unconnected-(U1-GND-Pad28) -> GND
- U1 pad 3: unconnected-(U1-GND-Pad3) -> GND
- U1 pad 31: unconnected-(U1-GPIO26_ADC0-Pad31) -> /MUX0_A
- U1 pad 32: unconnected-(U1-GPIO27_ADC1-Pad32) -> /MUX1_A
- U1 pad 33: unconnected-(U1-AGND-Pad33) -> GND
- U1 pad 36: unconnected-(U1-3V3-Pad36) -> /VDD33
- U1 pad 38: unconnected-(U1-GND-Pad38) -> GND
- U1 pad 4: unconnected-(U1-GPIO2-Pad4) -> /SCK
- U1 pad 40: unconnected-(U1-VBUS-Pad40) -> /VDD50
- U1 pad 42: unconnected-(U1-GND-Pad42) -> GND
- U1 pad 5: unconnected-(U1-GPIO3-Pad5) -> /MOSI
- U1 pad 6: unconnected-(U1-GPIO4-Pad6) -> /MISO
- U1 pad 7: unconnected-(U1-GPIO5-Pad7) -> /CS
- U1 pad 8: unconnected-(U1-GND-Pad8) -> GND
- U1 pad 9: unconnected-(U1-GPIO6-Pad9) -> /RST
- U2 pad 11: unconnected-(U2E-V--Pad11) -> GND
- U2 pad 4: unconnected-(U2E-V+-Pad4) -> /VDD50
- U3 pad 11: unconnected-(U3E-V--Pad11) -> GND
- U3 pad 4: unconnected-(U3E-V+-Pad4) -> /VDD33
- U4 pad 10: unconnected-(U4-S1-Pad10) -> /MUX0_S1
- U4 pad 11: unconnected-(U4-S0-Pad11) -> /MUX0_S0
- U4 pad 3: unconnected-(U4-A-Pad3) -> /MUX0_A
- U4 pad 6: unconnected-(U4-~{E}-Pad6) -> /MUX0_EB
- U4 pad 7: unconnected-(U4-VEE-Pad7) -> GND
- U4 pad 8: unconnected-(U4-GND-Pad8) -> GND
- U4 pad 9: unconnected-(U4-S2-Pad9) -> /MUX0_S2
- U5 pad 10: V33IN2 -> V33IN6
- U5 pad 11: unconnected-(U5E-V--Pad11) -> GND
- U5 pad 12: V33IN3 -> V33IN7
- U5 pad 13: /VBUFF6 -> /VBUFF7
- U5 pad 14: /VBUFF6 -> /VBUFF7
- U5 pad 3: V33IN0 -> V33IN4
- U5 pad 4: unconnected-(U5E-V+-Pad4) -> /VDD33
- U5 pad 5: V33IN1 -> V33IN5
- U6 pad 11: unconnected-(U6E-V--Pad11) -> GND
- U6 pad 4: unconnected-(U6E-V+-Pad4) -> /VDD50
- U7 pad 1: /VBUFF4 -> /Y+
- U7 pad 10: unconnected-(U7-S1-Pad10) -> /MUX1_S1
- U7 pad 11: unconnected-(U7-S0-Pad11) -> /MUX1_S0
- U7 pad 12: /VBUFF3 -> /VBUFF11
- U7 pad 13: /VBUFF0 -> /VBUFF8
- U7 pad 14: /VBUFF1 -> /VBUFF9
- U7 pad 2: /VBUFF6 -> /X-
- U7 pad 3: unconnected-(U7-A-Pad3) -> /MUX1_A
- U7 pad 4: /VBUFF7 -> /X+
- U7 pad 5: /VBUFF5 -> /Y-
- U7 pad 6: unconnected-(U7-~{E}-Pad6) -> /MUX1_EB
- U7 pad 7: unconnected-(U7-VEE-Pad7) -> GND
- U7 pad 8: unconnected-(U7-GND-Pad8) -> GND
- U7 pad 9: unconnected-(U7-S2-Pad9) -> /MUX1_S2
Routing:
- net +5V0: track 66.4 -> 0.00 mm
- net /VBUFF7: track 0.00 -> 62.8 mm, vias 0 -> 2
- net /VBUFF5: track 0.00 -> 61.7 mm
- net /VBUFF6: track 0.00 -> 53.7 mm, vias 0 -> 2
- net /X-: track 0.00 -> 53.1 mm
- net /VBUFF3: track 0.00 -> 51.8 mm, vias 0 -> 4
- net /VBUFF4: track 0.00 -> 49.6 mm
- net /Y+: track 0.00 -> 49.0 mm
- net /MUX0_A: track 0.00 -> 46.1 mm, vias 0 -> 2
- net /Y-: track 0.00 -> 45.3 mm
- net OUT4: track 44.4 -> 0.00 mm
- net OUT1: track 44.3 -> 0.00 mm
- net /MUX1_A: track 0.00 -> 43.0 mm, vias 0 -> 1
- net OUT2: track 43.0 -> 0.00 mm
- net OUT3: track 42.9 -> 0.00 mm
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- added copper zone on In2.Cu, net /VDD33
- added copper zone on F.Cu, net /VDD50
- removed copper zone on In2.Cu, net GND
Other:
- board size 79 x 45 mm -> 122.3 x 48.8 mm
- board text added: "EYEVOLT Ver.: 1.0"
- board text added: "Pins 1/2"
- board text removed: "+5V0"
- board text removed: "EXT VOLT"
- board text removed: "INPUT"
- board text removed: "OUT1"
- board text removed: "OUT2"
- board text removed: "OUT3"
- board text removed: "OUT4"
- board text removed: "OUT5"
- board text removed: "OUT6"
- board text removed: "OUT7"
- board text removed: "OUTPUT"
- board text removed: "VOLTAGE FOLLOWER Ver.: 1.0"
