File: hw/pcb/eyevolt.kicad_pcb (KiCad board)
At the start: 4 copper layers, 122.3 x 78.8 mm, 117 parts, among them J1 Conn_02x10_Odd_Even, J2 DAC_PWM_DAC_OUT_2x20, U1 Pico, U100 OPA316QDBVTQ1, U101 OPA316QDBVTQ1, U102 OPA316QDBVTQ1, U103 OPA316QDBVTQ1, U104 OPA316QDBVTQ1, U105 OPA316QDBVTQ1, U106 OPA316QDBVTQ1, U107 OPA316QDBVTQ1, U2 MCP6L04x-xSL, U3 MCP6L04x-xSL, U4 74HCT4051, U5 MCP6L04x-xSL, U6 MCP6L04x-xSL, U7 74HCT4051, U8 74HCT4051 DAC_FB_MUX

Commit message: cleaned schematic, component placement on layout
Parts:
- removed C170: 1uF, Capacitor_SMD:C_0805_2012Metric_Pad1.18x1.45mm_HandSolder
- removed R170, R171: 10k, Resistor_SMD:R_0805_2012Metric_Pad1.20x1.40mm_HandSolder
- removed R172: DNP 10k TH ALT, Resistor_THT:R_Axial_DIN0207_L6.3mm_D2.5mm_P7.62mm_Horizontal
- removed U107: OPA316QDBVTQ1, Package_TO_SOT_SMD:SOT-23-5
- added C9: 1uF, Capacitor_SMD:C_0805_2012Metric_Pad1.18x1.45mm_HandSolder, F.Cu at (133.6, 100.8)
- added R23: 10k, Resistor_SMD:R_0805_2012Metric_Pad1.20x1.40mm_HandSolder, F.Cu at (132.6, 107.0)
- added R7: 10k, Resistor_SMD:R_0805_2012Metric_Pad1.20x1.40mm_HandSolder, F.Cu at (132.6, 91.7)
- added R8: DNP 10k TH ALT, Resistor_THT:R_Axial_DIN0207_L6.3mm_D2.5mm_P7.62mm_Horizontal, F.Cu at (132.6, 87.8)
- added U7: OPA316QDBVTQ1, Package_TO_SOT_SMD:SOT-23-5, F.Cu at (10.8, 153.1)
- H1, H2, H3, H4: footprint MountingHole:MountingHole_3.2mm_M3 -> MountingHole:MountingHole_3.5mm_Pad_Via
- moved R45 175.0 mm to (-112.0, 127.6), turned to 180 degrees
- moved C44 171.4 mm to (-110.6, 121.7)
- moved U13 171.4 mm to (-112.0, 124.9)
- moved R46 171.2 mm to (-95.1, 128.5), turned to 180 degrees
- moved R47 169.4 mm to (-79.1, 129.2), turned to 180 degrees
- moved C45 167.6 mm to (-93.8, 122.6)
- moved U14 167.6 mm to (-95.1, 125.8)
- moved C46 165.7 mm to (-77.2, 123.3)
- moved U15 165.7 mm to (-79.1, 126.5)
- moved R48 163.4 mm to (-60.0, 130.4), turned to 180 degrees
- moved R25 162.3 mm to (-46.1, 132.1), turned to 180 degrees
- moved C47 159.8 mm to (-58.6, 124.6)
- moved U16 159.8 mm to (-60.0, 127.8)
- moved R26 159.6 mm to (-30.7, 133.0), turned to 180 degrees
- moved C20 158.7 mm to (-45.8, 125.7)
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- renumbered C5 to C1, C172 to C10, C141 to C11, C143 to C12, C151 to C13, C153 to C14, C161 to C15, C163 to C16, C171 to C17, C173 to C18, C4 to C19, C6 to C2, C144 to C20, C154 to C21, C164 to C22, C174 to C23, C3 to C24, C1 to C25, C2 to C26, C100 to C27, C102 to C28, C110 to C29, C140 to C3, C112 to C30, C120 to C31, C122 to C32, C130 to C33, C132 to C34, C101 to C35, C103 to C36, C111 to C37, C113 to C38, C121 to C39, C142 to C4, C123 to C40, C131 to C41, C133 to C42, C180 to C43, C104 to C44, C114 to C45, C124 to C46, C134 to C47, C150 to C5, C152 to C6, C160 to C7, C162 to C8, R140 to R1, R2 to R10, R3 to R11, R4 to R12, R5 to R13, R6 to R14, R7 to R15, R8 to R16, R141 to R17, R143 to R18, R151 to R19, R142 to R2, R153 to R20, R161 to R21, R163 to R22, R173 to R24, R144 to R25, R154 to R26, R164 to R27, R174 to R28, R100 to R29, R150 to R3, R102 to R30, R110 to R31, R112 to R32, R120 to R33, R122 to R34, R130 to R35, R132 to R36, R101 to R37, R103 to R38, R111 to R39, R152 to R4, R113 to R40, R121 to R41, R123 to R42, R131 to R43, R133 to R44, R104 to R45, R114 to R46, R124 to R47, R134 to R48, R160 to R5, R162 to R6, R1 to R9, U6 to U1, U7 to U10, U4 to U11, U8 to U12, U100 to U13, U101 to U14, U102 to U15, U103 to U16, U104 to U4, U105 to U5, U106 to U6, U5 to U8, U1 to U9
Connections:
- U9 pad 14: /MUX0_S0 -> /MUX0_S2
- U9 pad 16: /MUX0_S2 -> /MUX0_S0
Routing:
- net GND: track 155.7 -> 7.19 mm, vias 48 -> 4
- net /DAC_PWM7: track 131.9 -> 5.49 mm, vias 4 -> 0
- net /DAC_PWM6: track 119.1 -> 2.54 mm, vias 4 -> 0
- net /DAC_OUT6: track 113.6 -> 1.54 mm, vias 2 -> 1
- net /DAC_PWM5: track 113.0 -> 2.54 mm, vias 4 -> 0
- net /DAC_OUT7: track 110.8 -> 1.59 mm, vias 4 -> 1
- net /DAC_PWM4: track 110.2 -> 2.54 mm, vias 4 -> 0
- net /DAC_PWM3: track 103.9 -> 2.54 mm, vias 4 -> 0
- net /DAC_OUT5: track 94.7 -> 2.54 mm, vias 2 -> 1
- net (no net): track 89.1 -> 0.00 mm, vias 3 -> 0
- net /DAC_PWM2: track 88.6 -> 2.54 mm, vias 4 -> 0
- net /DAC_OUT4: track 88.3 -> 2.59 mm, vias 2 -> 1
- net /DAC_OUT2: track 81.5 -> 1.68 mm
- net /DAC_PWM1: track 75.2 -> 2.54 mm, vias 2 -> 0
- net /DAC_OUT0: track 71.8 -> 3.14 mm
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- added copper zone on F.Cu, net GND
- removed copper zone on F.Cu, net /VDD33
- removed copper zone on F.Cu, net /VDD50
Other:
- board size 122.3 x 78.8 mm -> 125 x 87 mm

Commit message: layout finished
Parts:
- C1, C19, C2, C24, C25, C26: footprint Capacitor_SMD:C_0805_2012Metric_Pad1.18x1.45mm_HandSolder -> Capacitor_SMD:C_0402_1005Metric_Pad0.74x0.62mm_HandSolder
- C20, C21, C22, C23, C43, C44, C45, C46, C47: footprint Capacitor_SMD:C_0805_2012Metric -> Capacitor_SMD:C_0402_1005Metric_Pad0.74x0.62mm_HandSolder
- moved R45 162.6 mm to (50.4, 119.2), turned to 0 degrees
- moved R46 158.5 mm to (63.2, 119.2), turned to 0 degrees
- moved U13 158.4 mm to (46.4, 120.3), turned to -90 degrees
- moved C44 156.8 mm to (46.2, 123.3), turned to 180 degrees
- moved R47 154.9 mm to (75.4, 119.3), turned to 0 degrees
- moved U14 154.0 mm to (58.8, 120.3), turned to -90 degrees
- moved C45 152.6 mm to (58.8, 123.5), turned to 180 degrees
- moved U15 150.5 mm to (71.2, 120.4), turned to -90 degrees
- moved C46 148.5 mm to (71.3, 123.5), turned to 180 degrees
- moved R48 148.3 mm to (87.9, 119.3), turned to 0 degrees
- moved R25 146.8 mm to (100.2, 119.3), turned to 0 degrees
- moved R26 144.2 mm to (112.8, 119.3), turned to 0 degrees
- moved U16 143.9 mm to (83.7, 120.4), turned to -90 degrees
- moved U4 142.5 mm to (96.1, 120.4), turned to -90 degrees
- moved C47 142.3 mm to (83.8, 123.5), turned to 180 degrees
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Connections:
- U9 pad 19: /DACMUX_S0 -> /DACMUX_S1
- U9 pad 20: /DACMUX_S1 -> /DACMUX_S0
- U9 pad 25: /MUX1_S2 -> /MUX1_S0
- U9 pad 27: /MUX1_S0 -> /MUX1_S2
Routing:
- net /VDD33: track 6.24 -> 407.2 mm, vias 2 -> 14
- net /VDD50: track 0.00 -> 234.4 mm, vias 0 -> 2
- net /DAC_PWM7: track 5.49 -> 176.0 mm
- net /DAC_PWM6: track 2.54 -> 152.7 mm
- net /DAC_PWM5: track 2.54 -> 132.1 mm
- net /DAC_OUT7: track 1.59 -> 128.6 mm, vias 1 -> 2
- net /DAC_OUT0: track 3.14 -> 118.4 mm
- net /DAC_PWM4: track 2.54 -> 115.2 mm
- net /DAC_OUT1: track 2.27 -> 107.1 mm
- net /DAC_OUT6: track 1.54 -> 103.3 mm, vias 1 -> 2
- net /DAC_OUT3: track 2.42 -> 101.1 mm
- net /DAC_PWM3: track 2.54 -> 100.4 mm
- net /DAC_OUT5: track 2.54 -> 95.2 mm, vias 1 -> 2
- net /DAC_OUT2: track 1.68 -> 89.3 mm
- net /DAC_OUT4: track 2.59 -> 88.0 mm, vias 1 -> 2
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- added copper zone on In2.Cu, net GND
- removed copper zone on In2.Cu, net /VDD33
Other:
- board size 125 x 87 mm -> 123.7 x 94 mm
- board text added: "+3V3"
- board text added: "+5V0"
- board text added: "OUT0"
- board text added: "OUT1"
- board text added: "OUT2"
- board text added: "OUT3"
- board text added: "OUT4"
- board text added: "OUT5"
- board text added: "OUT6"
- board text added: "OUT7"
- board text added: "PWM0"
- board text added: "PWM1"
- board text added: "PWM2"
- board text added: "PWM3"
- board text added: "PWM4"
- board text added: "PWM5"
- board text added: "PWM6"
- board text added: "PWM7"
- board text removed: "VDD50"
