File: hw/pcb/eyevolt.kicad_sch (KiCad schematic)
At the start: 16 parts, among them J1 Conn_02x10_Odd_Even, U1 Pico, U2 MCP6L04x-xSL, U3 MCP6L04x-xSL, U4 74HCT4051, U5 MCP6L04x-xSL, U6 MCP6L04x-xSL, U7 74HCT4051

Commit message: First version of PCB completed
Parts:
- added C1, C2, C3, C4, C5, C6: C, Capacitor_SMD:C_0805_2012Metric_Pad1.18x1.45mm_HandSolder, symbol Device:C
- added H1, H2, H3, H4: MountingHole_Pad, MountingHole:MountingHole_3.2mm_M3, symbol Mechanical:MountingHole_Pad
- added J2, J3: Conn_01x15, Connector_PinHeader_2.54mm:PinHeader_1x15_P2.54mm_Vertical, symbol Connector_Generic:Conn_01x15
- U4, U7: footprint Package_SO:SOIC-14_3.9x8.7mm_P1.27mm -> Package_SO:SOIC-16_3.9x9.9mm_P1.27mm
Connections:
- net GND: now also U1.13 (GND), U1.18 (GND), U1.23 (GND), U1.28 (GND), U1.3 (GND), U1.33 (AGND), U1.38 (GND), U1.42 (GND), U1.8 (GND), U2.11 (V-), U3.11 (V-), U4.7 (VEE), U4.8 (GND), U5.11 (V-), U6.11 (V-), U7.7 (VEE), U7.8 (GND), C1.2, C2.2, C3.2, C4.2, C5.2, C6.2, J2.2 (Pin_2), J3.2 (Pin_2)
- net V33IN0: no longer U5.3 (+)
- net V33IN1: no longer U5.5 (+)
- net V33IN2: no longer U5.10 (+)
- net V33IN3: no longer U5.12 (+)
- net V33IN4: now also U5.3 (+)
- net V33IN5: now also U5.5 (+)
- net V33IN6: now also U5.10 (+)
- net V33IN7: now also U5.12 (+)
- net VBUFF0: no longer U7.13 (A0)
- net VBUFF1: no longer U7.14 (A1)
- net VBUFF10: now also U7.15 (A2)
- net VBUFF11: now also U7.12 (A3)
- net VBUFF2: no longer U7.15 (A2)
- net VBUFF3: no longer U7.12 (A3)
- net VBUFF4: no longer U7.1 (A4)
- net VBUFF5: no longer U7.5 (A5)
- net VBUFF6: no longer U5.13 (-), U5.14, U7.2 (A6)
- net VBUFF7: now also U5.13 (-), U5.14; no longer U7.4 (A7)
- net VBUFF8: now also U7.13 (A0)
- net VBUFF9: now also U7.14 (A1)
- net MUX1_S1: now reaches U7.10 (S1)
- net MUX1_S1: now also U1.26 (GPIO20)
- net MUX1_S0: now reaches U7.11 (S0)
- net MUX1_S0: now also U1.27 (GPIO21)
- net VDD33: now reaches U7.16 (VCC)
- net VDD33: now also U1.36 (3V3), U3.4 (V+), U4.16 (VCC), U5.4 (V+), C1.1, C2.1, C3.1, C4.1
- net MUX1_A: now reaches U7.3 (A)
- net MUX1_A: now also U1.32 (GPIO27_ADC1)
- net MUX1_EB: now reaches U7.6 (~{E})
- net MUX1_EB: now also U1.24 (GPIO18)
- net MUX1_S2: now reaches U7.9 (S2)
- net MUX1_S2: now also U1.25 (GPIO19)
- net VDD50: now reaches U6.4 (V+)
- net VDD50: now also U1.40 (VBUS), U2.4 (V+), C5.1, C6.1, J2.1 (Pin_1), J3.1 (Pin_1)
- net WAIT: now reaches U1.10 (GPIO7)
- net WAIT: now also J2.10 (Pin_10), J3.10 (Pin_10)
- net INT: now reaches U1.11 (GPIO8)
- net INT: now also J2.11 (Pin_11), J3.11 (Pin_11)
- net MUX0_S0: now reaches U1.14 (GPIO10)
- net MUX0_S0: now also U4.11 (S0)
- net MUX0_S1: now reaches U1.15 (GPIO11)
- net MUX0_S1: now also U4.10 (S1)
- net MUX0_S2: now reaches U1.16 (GPIO12)
- net MUX0_S2: now also U4.9 (S2)
- net MUX0_EB: now reaches U1.17 (GPIO13)
- net MUX0_EB: now also U4.6 (~{E})
- net MUX0_A: now reaches U1.31 (GPIO26_ADC0)
- net MUX0_A: now also U4.3 (A)
- net SCK: now reaches U1.4 (GPIO2)
- net SCK: now also J2.5 (Pin_5), J3.5 (Pin_5)
- net MOSI: now reaches U1.5 (GPIO3)
- net MOSI: now also J2.7 (Pin_7), J3.7 (Pin_7)
- net MISO: now reaches U1.6 (GPIO4)
- net MISO: now also J2.6 (Pin_6), J3.6 (Pin_6)
- net CS: now reaches U1.7 (GPIO5)
- net CS: now also J2.8 (Pin_8), J3.8 (Pin_8)
- net RST: now reaches U1.9 (GPIO6)
- net RST: now also J2.9 (Pin_9), J3.9 (Pin_9)
- new net 3Vo: J2.3 (Pin_3), J3.3 (Pin_3)
- new net LITE: J2.4 (Pin_4), J3.4 (Pin_4)
- new net X+: J2.15 (Pin_15), J3.15 (Pin_15), U7.4 (A7)
- new net X-: J2.14 (Pin_14), J3.14 (Pin_14), U7.2 (A6)
- new net Y+: J2.12 (Pin_12), J3.12 (Pin_12), U7.1 (A4)
- new net Y-: J2.13 (Pin_13), J3.13 (Pin_13), U7.5 (A5)
- no-connect marks 0 -> 23
Other:
- title: (none) -> EYEVOLT

Commit message: Start new 2.0 version with 8 PWM-based DAC
Parts:
- removed J2, J3: Conn_01x15, Connector_PinHeader_2.54mm:PinHeader_1x15_P2.54mm_Vertical, symbol Connector_Generic:Conn_01x15
- added C100, C101, C110, C111, C120, C121, C130, C131, C140, C141, C150, C151, C160, C161, C170, C171: 1uF, Capacitor_SMD:C_0805_2012Metric_Pad1.18x1.45mm_HandSolder, symbol Device:C
- added C102, C103, C112, C113, C122, C123, C132, C133, C142, C143, C152, C153, C162, C163, C172, C173: DNP 1uF TH ALT, Capacitor_THT:C_Disc_D5.0mm_W2.5mm_P5.00mm, symbol Device:C
- added C104, C114, C124, C134, C144, C154, C164, C174, C180: 100nF, Capacitor_SMD:C_0805_2012Metric, symbol Device:C
- added J2: DAC_PWM_DAC_OUT_2x20, Connector_IDC:IDC-Header_2x20_P2.54mm_Horizontal, symbol Connector_Generic:Conn_02x20_Odd_Even
- added R100, R101, R110, R111, R120, R121, R130, R131, R140, R141, R150, R151, R160, R161, R170, R171: 10k, Resistor_SMD:R_0805_2012Metric_Pad1.20x1.40mm_HandSolder, symbol Device:R
- added R102, R103, R112, R113, R122, R123, R132, R133, R142, R143, R152, R153, R162, R163, R172, R173: DNP 10k TH ALT, Resistor_THT:R_Axial_DIN0207_L6.3mm_D2.5mm_P7.62mm_Horizontal, symbol Device:R
- added R104, R114, R124, R134, R144, R154, R164, R174: 0R OUT_LINK, Resistor_SMD:R_0805_2012Metric_Pad1.20x1.40mm_HandSolder, symbol Device:R
- added U100, U101, U102, U103, U104, U105, U106, U107: OPA316QDBVTQ1, Package_TO_SOT_SMD:SOT-23-5, symbol Amplifier_Operational:MCP6001-OT
- added U8: 74HCT4051 DAC_FB_MUX, Package_SO:SOIC-16_3.9x9.9mm_P1.27mm, symbol 74xx:74HCT4051
Connections:
- net V55IN0 is gone; now on net V50IN0: J1.2 (Pin_2)
- net V55IN1 is gone; now on net V50IN1: J1.4 (Pin_4)
- net V55IN2 is gone; now on net V50IN2: J1.6 (Pin_6)
- net V55IN3 is gone; now on net V50IN3: J1.8 (Pin_8)
- net GND: now also C100.2, C101.2, C102.2, C103.2, C104.2, C110.2, C111.2, C112.2, C113.2, C114.2, C120.2, C121.2, C122.2, C123.2, C124.2, C130.2, C131.2, C132.2, C133.2, C134.2, C140.2, C141.2, C142.2, C143.2, C144.2, C150.2, C151.2, C152.2, C153.2, C154.2, C160.2, C161.2, C162.2, C163.2, C164.2, C170.2, C171.2, C172.2, C173.2, C174.2, C180.2, J2.1 (Pin_1), J2.2 (Pin_2), J2.3 (Pin_3), J2.4 (Pin_4), U100.2 (V-), U101.2 (V-), U102.2 (V-), U103.2 (V-), U104.2 (V-), U105.2 (V-), U106.2 (V-), U107.2 (V-), U8.7 (VEE), U8.8 (GND)
- net VDD33: now also C104.1, C114.1, C124.1, C134.1, C144.1, C154.1, C164.1, C174.1, C180.1, J2.7 (Pin_7), J2.8 (Pin_8), U100.5 (V+), U101.5 (V+), U102.5 (V+), U103.5 (V+), U104.5 (V+), U105.5 (V+), U106.5 (V+), U107.5 (V+), U8.16 (VCC)
- net VDD50: now also J2.5 (Pin_5), J2.6 (Pin_6)
- net DAC_PWM7: now reaches U1.12 (GPIO9)
- net DAC_PWM7: now also J2.25 (Pin_25), J2.26 (Pin_26), R170.1, R172.1
- net DACMUX_S0: now reaches U1.19 (GPIO14)
- net DACMUX_S0: now also U8.11 (S0)
- net DACMUX_S1: now reaches U1.20 (GPIO15)
- net DACMUX_S1: now also U8.10 (S1)
- net DACMUX_S2: now reaches U1.21 (GPIO16)
- net DACMUX_S2: now also U8.9 (S2)
- net DACMUX_EB: now reaches U1.22 (GPIO17)
- net DACMUX_EB: now also U8.6 (~{E})
- net CS renamed DAC_PWM3
- net DAC_PWM3: now also J2.33 (Pin_33), J2.34 (Pin_34), R130.1, R132.1
- net INT renamed DAC_PWM6
- net DAC_PWM6: now also J2.27 (Pin_27), J2.28 (Pin_28), R160.1, R162.1
- net MISO renamed DAC_PWM2
- net DAC_PWM2: now also J2.35 (Pin_35), J2.36 (Pin_36), R120.1, R122.1
- net MOSI renamed DAC_PWM1
- net DAC_PWM1: now also J2.37 (Pin_37), J2.38 (Pin_38), R110.1, R112.1
- net MUX0_A renamed MON_ADC_A
- net MON_ADC_A: now also U7.3 (A); no longer U4.3 (A)
- net MUX1_A renamed DAC_FB_A
- net DAC_FB_A: now also U8.3 (A); no longer U7.3 (A)
- net RST renamed DAC_PWM4
- net DAC_PWM4: now also J2.31 (Pin_31), J2.32 (Pin_32), R140.1, R142.1
- net SCK renamed DAC_PWM0
- net DAC_PWM0: now also J2.39 (Pin_39), J2.40 (Pin_40), R100.1, R102.1
- net WAIT renamed DAC_PWM5
- net DAC_PWM5: now also J2.29 (Pin_29), J2.30 (Pin_30), R150.1, R152.1
- net X+ renamed MUX1_SPARE_A7
- net X- renamed MUX1_SPARE_A6
- net Y+ renamed MUX0_A_TO_MUX1
- net MUX0_A_TO_MUX1: now also U4.3 (A)
- net Y- renamed MUX1_SPARE_A5
- new net DAC0_BUF: R104.1, U100.1, U100.4 (-)
- new net DAC0_FILT: C101.1, C103.1, R101.2, R103.2, U100.3 (+)
- new net DAC0_RC1: C100.1, C102.1, R100.2, R101.1, R102.2, R103.1
- new net DAC1_BUF: R114.1, U101.1, U101.4 (-)
- new net DAC1_FILT: C111.1, C113.1, R111.2, R113.2, U101.3 (+)
- new net DAC1_RC1: C110.1, C112.1, R110.2, R111.1, R112.2, R113.1
- new net DAC2_BUF: R124.1, U102.1, U102.4 (-)
- new net DAC2_FILT: C121.1, C123.1, R121.2, R123.2, U102.3 (+)
- new net DAC2_RC1: C120.1, C122.1, R120.2, R121.1, R122.2, R123.1
- new net DAC3_BUF: R134.1, U103.1, U103.4 (-)
- new net DAC3_FILT: C131.1, C133.1, R131.2, R133.2, U103.3 (+)
- new net DAC3_RC1: C130.1, C132.1, R130.2, R131.1, R132.2, R133.1
- new net DAC4_BUF: R144.1, U104.1, U104.4 (-)
- new net DAC4_FILT: C141.1, C143.1, R141.2, R143.2, U104.3 (+)
- new net DAC4_RC1: C140.1, C142.1, R140.2, R141.1, R142.2, R143.1
- new net DAC5_BUF: R154.1, U105.1, U105.4 (-)
- new net DAC5_FILT: C151.1, C153.1, R151.2, R153.2, U105.3 (+)
- new net DAC5_RC1: C150.1, C152.1, R150.2, R151.1, R152.2, R153.1
- new net DAC6_BUF: R164.1, U106.1, U106.4 (-)
- new net DAC6_FILT: C161.1, C163.1, R161.2, R163.2, U106.3 (+)
- new net DAC6_RC1: C160.1, C162.1, R160.2, R161.1, R162.2, R163.1
- new net DAC7_BUF: R174.1, U107.1, U107.4 (-)
- new net DAC7_FILT: C171.1, C173.1, R171.2, R173.2, U107.3 (+)
- new net DAC7_RC1: C170.1, C172.1, R170.2, R171.1, R172.2, R173.1
- new net DAC_OUT0: J2.23 (Pin_23), J2.24 (Pin_24), R104.2, U8.13 (A0)
- new net DAC_OUT1: J2.21 (Pin_21), J2.22 (Pin_22), R114.2, U8.14 (A1)
- new net DAC_OUT2: J2.19 (Pin_19), J2.20 (Pin_20), R124.2, U8.15 (A2)
- new net DAC_OUT3: J2.17 (Pin_17), J2.18 (Pin_18), R134.2, U8.12 (A3)
- new net DAC_OUT4: J2.15 (Pin_15), J2.16 (Pin_16), R144.2, U8.1 (A4)
- new net DAC_OUT5: J2.13 (Pin_13), J2.14 (Pin_14), R154.2, U8.5 (A5)
- new net DAC_OUT6: J2.11 (Pin_11), J2.12 (Pin_12), R164.2, U8.2 (A6)
- new net DAC_OUT7: J2.10 (Pin_10), J2.9 (Pin_9), R174.2, U8.4 (A7)
Other:
- note added: "8x PWM DAC: GPIO2-GPIO9 -> 2-pole RC -> OPA316 -> J2. 10-20mA max per output; not all at max together."
- note added: "ADC mux: U4 -> U7 A4 -> GPIO26_ADC0. U8 feeds DAC_OUT0..7 to GPIO27_ADC1."
