File: hw/pcb/eyevolt.kicad_sch (KiCad schematic)
At the start: 117 parts, among them J1 Conn_02x10_Odd_Even, J2 DAC_PWM_DAC_OUT_2x20, U1 Pico, U100 OPA316QDBVTQ1, U101 OPA316QDBVTQ1, U102 OPA316QDBVTQ1, U103 OPA316QDBVTQ1, U104 OPA316QDBVTQ1, U105 OPA316QDBVTQ1, U106 OPA316QDBVTQ1, U107 OPA316QDBVTQ1, U2 MCP6L04x-xSL, U3 MCP6L04x-xSL, U4 74HCT4051, U5 MCP6L04x-xSL, U6 MCP6L04x-xSL, U7 74HCT4051, U8 74HCT4051 DAC_FB_MUX

Commit message: cleaned schematic, component placement on layout
Parts:
- H1, H2, H3, H4: footprint MountingHole:MountingHole_3.2mm_M3 -> MountingHole:MountingHole_3.5mm_Pad_Via
- renumbered C5 to C1, C172 to C10, C141 to C11, C143 to C12, C151 to C13, C153 to C14, C161 to C15, C163 to C16, C171 to C17, C173 to C18, C4 to C19, C6 to C2, C144 to C20, C154 to C21, C164 to C22, C174 to C23, C3 to C24, C1 to C25, C2 to C26, C100 to C27, C102 to C28, C110 to C29, C140 to C3, C112 to C30, C120 to C31, C122 to C32, C130 to C33, C132 to C34, C101 to C35, C103 to C36, C111 to C37, C113 to C38, C121 to C39, C142 to C4, C123 to C40, C131 to C41, C133 to C42, C180 to C43, C104 to C44, C114 to C45, C124 to C46, C134 to C47, C150 to C5, C152 to C6, C160 to C7, C162 to C8, C170 to C9, R140 to R1, R2 to R10, R3 to R11, R4 to R12, R5 to R13, R6 to R14, R7 to R15, R8 to R16, R141 to R17, R143 to R18, R151 to R19, R142 to R2, R153 to R20, R161 to R21, R163 to R22, R171 to R23, R173 to R24, R144 to R25, R154 to R26, R164 to R27, R174 to R28, R100 to R29, R150 to R3, R102 to R30, R110 to R31, R112 to R32, R120 to R33, R122 to R34, R130 to R35, R132 to R36, R101 to R37, R103 to R38, R111 to R39, R152 to R4, R113 to R40, R121 to R41, R123 to R42, R131 to R43, R133 to R44, R104 to R45, R114 to R46, R124 to R47, R134 to R48, R160 to R5, R162 to R6, R170 to R7, R172 to R8, R1 to R9, U6 to U1, U7 to U10, U4 to U11, U8 to U12, U100 to U13, U101 to U14, U102 to U15, U103 to U16, U104 to U4, U105 to U5, U106 to U6, U107 to U7, U5 to U8, U1 to U9
Connections:
- net GND: now also H1.1, H2.1, H3.1, H4.1
- net MUX0_S0: now also U9.16 (GPIO12); no longer U9.14 (GPIO10)
- net MUX0_S2: now also U9.14 (GPIO10); no longer U9.16 (GPIO12)
- no-connect marks 23 -> 14
Other:
- moved on the sheet: C1, C10, C11, C12, C13, C14, C15, C16, C17, C18, C19, C2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
